File: PCB/HDMI_SWITCH.kicad_sch (KiCad schematic)
At the start: 21 parts, among them J1 HDMI_A, J2 HDMI_A, J3 HDMI_A, SW1 SW_SPDT, U1 TMDS261BPAG, U2 24LC02, U3 74HC04, U4 AMS1117-3.3

Commit message: Add files via upload
Parts:
- removed U3: 74HC04, Package_SO:SOIC-14_3.9x8.7mm_P1.27mm, symbol 74xx:74HC04
Connections:
- net +3.3V: now also R6.2
- net GND: now also D2.1 (K), U2.7 (WP); no longer D1.1 (K)
- net S1: now also D1.1 (K); no longer R6.1
- net at J2.15 (SCL), U1.37 (SCL1): now also R1.2
- net at J2.16 (SDA), U1.36 (SDA1): no longer R1.2
- net at D1.2 (A): now also R6.1; no longer R6.2
- no-connect marks 25 -> 24
Other:
- moved on the sheet: D1, D2, R1, R6, R7
