File: PCB/HDMI_SWITCH.kicad_pcb (KiCad board)
At the start: 4 copper layers, 37.5 x 36.5 mm, 21 parts, among them J1 HDMI_A, J2 HDMI_A, J3 HDMI_A, SW1 SW_SPDT, U1 TMDS261BPAG, U2 24LC02, U3 74HC04, U4 AMS1117-3.3

Commit message: Add files via upload
Parts:
- removed U3: 74HC04, Package_SO:SOIC-14_3.9x8.7mm_P1.27mm
- moved R6 3.79 mm to (129.1, 56.3), turned to 180 degrees
- moved SW1 1.88 mm to (109.4, 46.2)
- moved H2 1.56 mm to (132.9, 49.4)
Connections:
- D1 pad 1: GND -> S1
- D2 pad 1: Net-(D2-K) -> GND
- R1 pad 2: Net-(J2-SDA) -> Net-(J2-SCL)
- R6 pad 1: S1 -> Net-(D1-A)
- R6 pad 2: Net-(D1-A) -> +3.3V
- U2 pad 7: unconnected-(U2-WP-Pad7) -> GND
Routing:
- net +3.3V: track 106.6 -> 116.7 mm, vias 2 -> 3
- net Net-(J2-SCL): track 6.39 -> 15.9 mm, vias 0 -> 2
- net S1: track 40.3 -> 45.7 mm, vias 3 -> 4
- net Net-(D2-K): track 3.84 -> 0.00 mm
- net Net-(D1-A): track 2.60 -> 1.54 mm
- net GND: track 103.8 -> 104.8 mm
- net Net-(J2-SDA): track 7.30 -> 6.39 mm
- added copper zone on In2.Cu, net +3.3V
Other:
- board size 37.5 x 36.5 mm -> 39 x 37 mm

Commit message: Add files via upload
Routing:
- net +3.3V: track 116.7 -> 127.2 mm, vias 3 -> 9
Changed lines of the file:
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@@
+	)
+	(segment
+		(start 119.8 59.75)
+		(end 119.35 60.2)
+		(width 0.6)
+		(layer "F.Cu")
+		(net 38)
 	)
 	(segment
@@
 	)
 	(segment
+		(start 121.2981 62.1019)
+		(end 120.35 63.05)
+		(width 0.6)
+		(layer "F.Cu")
+		(net 38)
+	)
+	(segment
 		(start 125.05 58.749999)
 		(end 122.750001 58.749999)
@@
 	)
 	(segment
-		(start 124.4481 64.5519)
+		(start 124.2231 64.3269)
 		(end 123.6981 63.8019)
+		(width 0.6)
+		(layer "F.Cu")
+		(net 38)
+	)
+	(segment
+		(start 121.675 58.325)
+		(end 120.775735 57.425735)
 		(width 0.6)
 		(layer "F.Cu")
@@
 	)
 	(segment
+		(start 124.2231 64.3269)
+		(end 124.2231 63.1269)
+		(width 0.6)
+		(layer "F.Cu")
+		(net 38)
+	)
+	(segment
 		(start 107 49.702)
 		(end 109.047001 51.749001)
@@
 	)
 	(segment
-		(start 121 60.5)
+		(start 121 59.75)
 		(end 121 59)
 		(width 0.6)
@@
 	)
 	(segment
+		(start 121 61.1038)
+		(end 120.3038 61.8)
+		(width 0.6)
+		(layer "F.Cu")
+		(net 38)
+	)
+	(segment
 		(start 112 74)
 		(end 112.801 74.801)
@@
 	)
 	(segment
+		(start 119.75 57.75)
+		(end 119.5 57.5)
+		(width 0.6)
+		(layer "F.Cu")
+		(net 38)
+	)
+	(segment
 		(start 123.3962 63.5)
 		(end 122 63.5)
@@
 	(segment
 		(start 121 59)
-		(end 119.5 57.5)
+		(end 119.75 57.75)
 		(width 0.6)
 		(layer "F.Cu")
@@
 	)
 	(segment
+		(start 120.3038 61.8)
+		(end 119.8 61.8)
+		(width 0.6)
+		(layer "F.Cu")
+		(net 38)
+	)
+	(segment
 		(start 109.899 52.748943)
 		(end 109.899 51.850001)
@@
 	)
 	(segment
+		(start 121.9981 62.1019)
+		(end 121.2981 62.1019)
+		(width 0.6)
+		(layer "F.Cu")
+		(net 38)
+	)
+	(segment
 		(start 112 73.5)
 		(end 110.4 71.9)
@@
 	(segment
 		(start 122.9481 63.0519)
-		(end 121 61.1038)
+		(end 121.9981 62.1019)
+		(width 0.6)
+		(layer "F.Cu")
+		(net 38)
+	)
+	(segment
+		(start 119.65 57.65)
+		(end 118.65 57.65)
+		(width 0.6)
+		(layer "F.Cu")
+		(net 38)
+	)
+	(segment
+		(start 124.2231 63.1269)
+		(end 124.65 62.7)
 		(width 0.6)
 		(layer "F.Cu")
@@
 	)
 	(segment
+		(start 119.75 57.75)
+		(end 119.65 57.65)
+		(width 0.6)
+		(layer "F.Cu")
+		(net 38)
+	)
+	(segment
+		(start 120.775735 57.425735)
+		(end 120.775735 56.875735)
+		(width 0.6)
+		(layer "F.Cu")
+		(net 38)
+	)
+	(segment
 		(start 120.75 64.75)
 		(end 122 63.5)
@@
 	)
 	(segment
+		(start 118.65 57.65)
+		(end 118.4 57.9)
+		(width 0.6)
+		(layer "F.Cu")
+		(net 38)
+	)
+	(segment
+		(start 124.4481 64.5519)
+		(end 124.2231 64.3269)
+		(width 0.6)
+		(layer "F.Cu")
+		(net 38)
+	)
+	(segment
 		(start 111.600056 54.449999)
 		(end 109.899 52.748943)
@@
 	)
 	(segment
+		(start 121.675 58.325)
+		(end 122.25 57.75)
+		(width 0.6)
+		(layer "F.Cu")
+		(net 38)
+	)
+	(segment
+		(start 121.9981 62.1019)
+		(end 121 61.1038)
+		(width 0.6)
+		(layer "F.Cu")
+		(net 38)
+	)
+	(segment
 		(start 109.047001 51.749001)
 		(end 110 51.749001)
@@
 	)
 	(segment
+		(start 121 60.5)
+		(end 121 59.75)
+		(width 0.6)
+		(layer "F.Cu")
+		(net 38)
+	)
+	(segment
 		(start 119.250001 55.38025)
 		(end 119.250001 57.250001)
@@
 	)
 	(segment
+		(start 121 59.75)
+		(end 119.8 59.75)
+		(width 0.6)
+		(layer "F.Cu")
+		(net 38)
+	)
+	(segment
 		(start 126.61975 58.749999)
 		(end 125.05 58.749999)
@@
 	(segment
 		(start 121 59)
-		(end 122.25 57.75)
+		(end 121.675 58.325)
 		(width 0.6)
 		(layer "F.Cu")
@@
 	(via
 		(at 113.676527 55.823472)
+		(size 0.6)
+		(drill 0.3)
+		(layers "F.Cu" "B.Cu")
+		(net 38)
+	)
+	(via
+		(at 120.35 63.05)
+		(size 0.6)
+		(drill 0.3)
+		(layers "F.Cu" "B.Cu")
+		(net 38)
+	)
+	(via
+		(at 119.8 61.8)
+		(size 0.6)
+		(drill 0.3)
+		(layers "F.Cu" "B.Cu")
+		(net 38)
+	)
+	(via
+		(at 119.35 60.2)
+		(size 0.6)
+		(drill 0.3)
+		(layers "F.Cu" "B.Cu")
+		(net 38)
+	)
+	(via
+		(at 120.775735 56.875735)
 		(size 0.6)
 		(drill 0.3)
@@
 		(size 0.6)
 		(drill 0.3)
+		(layers "F.Cu" "B.Cu")
+		(net 38)
+	)
+	(via
+		(at 118.4 57.9)
+		(size 0.6)
+		(drill 0.3)
+		(layers "F.Cu" "B.Cu")
+		(net 38)
+	)
+	(via
+		(at 124.65 62.7)
+		(size 0.6)
+		(drill 0.3)
